File: schematic/ECU.brd (EAGLE design)
At the start: 25 x 79 mm, 21 parts, among them J1 Break, J2 COMM, J3 PWS, J4 DISPLAY, J5 THROTTLE, J6 LED, J7 SPEED, Q1 NMOSFETSOT23, Q5 NMOSFETSOT23

Commit message: Fix stop sensor schematics
- Make stop sensor LOW by default, connected to GND.
- Add control transistor for break on BLDC
Connections:
- removed net STOUT: J1.2, J2.4, R3.1
- net 5V: now also J1.2
- net ST: now also J2.4, R3.1
Routing:
- net 5V: track 50.8 -> 83.6 mm, vias 1 -> 2
- net ST: track 20.1 -> 33.6 mm
- net STOUT: track 12.5 -> 0.00 mm
Changed lines of the file:
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@@
 <wire x1="6.2571" y1="52.8" x2="8.7571" y2="50.3" width="0.8128" layer="16"/>
 <wire x1="8.7571" y1="50.3" x2="8.7571" y2="49.8" width="0.8128" layer="16"/>
+<contactref element="J1" pad="2"/>
+<wire x1="8.7571" y1="49.8" x2="10.4571" y2="51.5" width="0.8128" layer="1"/>
+<wire x1="10.4571" y1="51.5" x2="14" y2="51.5" width="0.8128" layer="1"/>
+<via x="14" y="51.5" extent="1-16" drill="0.35"/>
+<wire x1="14" y1="51.5" x2="18.5" y2="47" width="0.8128" layer="16"/>
+<wire x1="18.5" y1="27.68" x2="19.32" y2="26.86" width="0.8128" layer="16"/>
+<wire x1="18.5" y1="47" x2="18.5" y2="27.68" width="0.8128" layer="16"/>
 </signal>
 <signal name="THIN">
@@
 <wire x1="21.09" y1="44.64" x2="22.19" y2="44.64" width="0.8128" layer="1"/>
 <wire x1="20.05" y1="29.67" x2="20.05" y2="43.6" width="0.8128" layer="1"/>
+<contactref element="J2" pad="4"/>
+<wire x1="20.3" y1="16.7" x2="21.86" y2="16.7" width="0.8128" layer="16"/>
+<wire x1="18.922" y1="18.078" x2="20.3" y2="16.7" width="0.8128" layer="16"/>
+<contactref element="R3" pad="1"/>
+<wire x1="18.922" y1="23.922" x2="18.922" y2="18.5" width="0.8128" layer="16"/>
+<wire x1="21.86" y1="26.86" x2="18.922" y2="23.922" width="0.8128" layer="16"/>
+<wire x1="18.922" y1="18.5" x2="18.922" y2="18.078" width="0.8128" layer="16"/>
 </signal>
 <signal name="BTN">
@@
 <contactref element="U$2" pad="19"/>
 </signal>
-<signal name="STOUT">
-<contactref element="J1" pad="2"/>
-<contactref element="J2" pad="4"/>
-<wire x1="19.32" y1="26.86" x2="19.32" y2="18.5" width="0.8128" layer="16"/>
-<wire x1="19.32" y1="18.5" x2="19.32" y2="17.68" width="0.8128" layer="16"/>
-<wire x1="20.3" y1="16.7" x2="21.86" y2="16.7" width="0.8128" layer="16"/>
-<wire x1="19.32" y1="17.68" x2="20.3" y2="16.7" width="0.8128" layer="16"/>
-<contactref element="R3" pad="1"/>
-<wire x1="18.922" y1="18.5" x2="19.32" y2="18.5" width="0.8128" layer="16"/>
-</signal>
 </signals>
