File: schematic/regulator.brd (EAGLE design)
At the start: 62 x 43 mm, 26 parts, among them J1 COMM, J2 STOP_LIGHT, J3 ON/OFF, J4 BATTERY, J5 DRIVER, J6 DRIVER POWER, Q1 NMOSFETSOT23, Q2 NMOSFETSOT23, Q3 NMOSFETSOT23, Q4 IRFR3607PBF

Commit message: Fix regulator schematics
- Fix regulator schematics, add missed voltage controll resistors
- Fix deprecated warnings for display
Parts:
- added R10, R9: 47K, eagle-ltspice:R1206
- added R11: 10K, eagle-ltspice:R1206
Connections:
- new net N$6: R10.1, R9.2
- new net N$9: R10.2, R11.1, U$1.4
- net 12V: now also R9.1; no longer U$1.4
- net GND: now also R11.2
Routing:
- net 12V: track 41.2 -> 35.0 mm
- net N$9: track 0.00 -> 4.82 mm
- net N$6: track 0.00 -> 2.54 mm
Changed lines of the file:
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@@
 <attribute name="VALUE" x="21.59" y="41.91" size="1.2" layer="28" ratio="10" rot="MR270"/>
+</element>
+<element name="R9" library="eagle-ltspice" library_urn="urn:adsk.eagle:library:217" package="R1206" package3d_urn="urn:adsk.eagle:package:13301/1" value="47K" x="38.1" y="26.67" smashed="yes" rot="R90">
+<attribute name="NAME" x="38.1" y="29.21" size="1.27" layer="25" rot="R90"/>
+<attribute name="SPICEMODEL" value="NONE" x="38.1" y="26.67" size="1.778" layer="27" rot="R90" display="off"/>
+<attribute name="SPICEPREFIX" value="R" x="38.1" y="26.67" size="1.778" layer="27" rot="R90" display="off"/>
+<attribute name="VALUE" x="39.37" y="25.4" size="1.27" layer="27" rot="R90"/>
+</element>
+<element name="R10" library="eagle-ltspice" library_urn="urn:adsk.eagle:library:217" package="R1206" package3d_urn="urn:adsk.eagle:package:13301/1" value="47K" x="35.56" y="26.67" smashed="yes" rot="R270">
+<attribute name="NAME" x="35.56" y="29.21" size="1.27" layer="25" rot="R90"/>
+<attribute name="SPICEMODEL" value="NONE" x="35.56" y="26.67" size="1.778" layer="27" rot="R270" display="off"/>
+<attribute name="SPICEPREFIX" value="R" x="35.56" y="26.67" size="1.778" layer="27" rot="R270" display="off"/>
+<attribute name="VALUE" x="34.29" y="27.94" size="1.27" layer="27" rot="R270"/>
+</element>
+<element name="R11" library="eagle-ltspice" library_urn="urn:adsk.eagle:library:217" package="R1206" package3d_urn="urn:adsk.eagle:package:13301/1" value="10K" x="33.02" y="26.67" smashed="yes" rot="R90">
+<attribute name="NAME" x="33.02" y="29.21" size="1.27" layer="25" rot="R90"/>
+<attribute name="SPICEMODEL" value="NONE" x="33.02" y="26.67" size="1.778" layer="27" rot="R90" display="off"/>
+<attribute name="SPICEPREFIX" value="R" x="33.02" y="26.67" size="1.778" layer="27" rot="R90" display="off"/>
+<attribute name="VALUE" x="33.02" y="25.4" size="1.27" layer="27" rot="R90"/>
 </element>
 </elements>
@@
 <via x="45.72" y="19.05" extent="1-16" drill="0.35"/>
 <via x="44.45" y="20.32" extent="1-16" drill="0.35"/>
-<via x="43.18" y="24.13" extent="1-16" drill="0.35"/>
-<via x="41.91" y="25.4" extent="1-16" drill="0.35"/>
+<via x="44.45" y="25.4" extent="1-16" drill="0.35"/>
+<via x="43.18" y="26.67" extent="1-16" drill="0.35"/>
 <via x="44.45" y="22.86" extent="1-16" drill="0.35"/>
-<via x="40.64" y="26.67" extent="1-16" drill="0.35"/>
+<via x="41.91" y="27.94" extent="1-16" drill="0.35"/>
 <contactref element="R6" pad="2"/>
 <contactref element="R7" pad="1"/>
@@
 <contactref element="J4" pad="GND"/>
 <contactref element="Q4" pad="2"/>
-<via x="39.37" y="27.94" extent="1-16" drill="0.35"/>
+<via x="40.64" y="29.21" extent="1-16" drill="0.35"/>
 <via x="22.86" y="30.48" extent="1-16" drill="0.35"/>
 <via x="26.67" y="16.51" extent="1-16" drill="0.35"/>
@@
 <via x="34.29" y="30.48" extent="1-16" drill="0.35"/>
 <via x="36.83" y="30.48" extent="1-16" drill="0.35"/>
-<via x="38.1" y="29.21" extent="1-16" drill="0.35"/>
+<via x="39.37" y="30.48" extent="1-16" drill="0.35"/>
 <via x="38.1" y="12.7" extent="1-16" drill="0.35"/>
 <via x="41.91" y="3.81" extent="1-16" drill="0.35"/>
@@
 <via x="19.05" y="3.81" extent="1-16" drill="0.35"/>
 <via x="10.16" y="8.89" extent="1-16" drill="0.35"/>
+<contactref element="R11" pad="2"/>
 </signal>
 <signal name="VIN">
@@
 <contactref element="J1" pad="1"/>
 <contactref element="D2" pad="1"/>
-<contactref element="U$1" pad="4"/>
-<wire x1="40.64" y1="13.97" x2="43.18" y2="11.43" width="1.27" layer="1"/>
 <wire x1="43.18" y1="11.43" x2="44.345" y2="11.43" width="1.27" layer="1"/>
 <wire x1="53.0912" y1="8.45" x2="52.07" y2="9.4712" width="1.27" layer="1"/>
@@
 <wire x1="46.3038" y1="9.4712" x2="44.345" y2="11.43" width="1.27" layer="1"/>
 <wire x1="46.3038" y1="9.4712" x2="49.53" y2="9.4712" width="1.27" layer="1"/>
-<wire x1="30.8" y1="25.4" x2="36.83" y2="25.4" width="1.27" layer="1"/>
-<wire x1="36.83" y1="25.4" x2="40.64" y2="21.59" width="1.27" layer="1"/>
-<wire x1="40.64" y1="21.59" x2="40.64" y2="13.97" width="1.27" layer="1"/>
+<contactref element="R9" pad="1"/>
+<wire x1="38.1" y1="25.248" x2="38.1" y2="23.978" width="0.8128" layer="1"/>
+<wire x1="44.345" y1="17.733" x2="38.1" y2="23.978" width="0.8128" layer="1"/>
+<wire x1="44.345" y1="17.733" x2="44.345" y2="11.43" width="0.8128" layer="1"/>
 </signal>
 <signal name="N$4">
@@
 <wire x1="10.19" y1="38.1" x2="8.89" y2="38.1" width="2.54" layer="16"/>
 </signal>
+<signal name="N$6">
+<contactref element="R10" pad="1"/>
+<contactref element="R9" pad="2"/>
+<wire x1="35.56" y1="28.092" x2="38.1" y2="28.092" width="0.8128" layer="1"/>
+</signal>
+<signal name="N$9">
+<contactref element="U$1" pad="4"/>
+<contactref element="R11" pad="1"/>
+<contactref element="R10" pad="2"/>
+<wire x1="30.8" y1="25.4" x2="32.868" y2="25.4" width="0.8128" layer="1"/>
+<wire x1="32.868" y1="25.4" x2="33.02" y2="25.248" width="0.8128" layer="1"/>
+<wire x1="33.02" y1="25.248" x2="35.56" y2="25.248" width="0.8128" layer="1"/>
+</signal>
 </signals>
